File: d2-motherboard-pcb/d2-motherboard-pcb.kicad_sch (KiCad schematic)
At the start: 31 parts, among them J1 FTDI, J2 Conn_01x02_Male, J3 Conn_01x02_Male, J4 Conn_01x04_Male, U1 PIC32CM6408MC00032-I/PT

Commit message: add debug board
Parts:
- removed J1: FTDI, Connector_PinHeader_2.54mm:PinHeader_1x06_P2.54mm_Vertical, symbol Connector:Conn_01x06_Male
- removed J3: Conn_01x02_Male, Connector_PinHeader_2.54mm:PinHeader_1x02_P2.54mm_Vertical, symbol Connector:Conn_01x02_Male
- removed R16: 0, Resistor_SMD:R_0603_1608Metric, symbol Device:R
- removed SWD1: Conn_02x05_Odd_Even, Connector_PinHeader_1.27mm:PinHeader_2x05_P1.27mm_Vertical, symbol Connector_Generic:Conn_02x05_Odd_Even
- removed TP1, TP2, TP5: TestPoint, Connector_PinHeader_2.54mm:PinHeader_1x01_P2.54mm_Vertical, symbol Connector:TestPoint
- added C22: 1uF, Capacitor_SMD:C_0603_1608Metric, symbol Device:C
- added C23: 10uF, Capacitor_SMD:C_1206_3216Metric_Pad1.33x1.80mm_HandSolder, symbol Device:C
- added C24: 22uF, Capacitor_SMD:C_0805_2012Metric_Pad1.18x1.45mm_HandSolder, symbol Device:C
- C4: footprint Capacitor_THT:CP_Radial_D5.0mm_P2.50mm -> Capacitor_THT:CP_Radial_D8.0mm_P3.50mm
- C6: value 47uF -> 0.1uF; footprint Capacitor_THT:CP_Radial_D5.0mm_P2.50mm -> Capacitor_SMD:C_0603_1608Metric
Connections:
- net +5V: now also C6.2, C22.2, C23.2, C24.1; no longer C6.1
- net FTDI_RXI_CONN: now also SWD3.7 (Pin_7); no longer SWD3.5 (Pin_5)
- net FTDI_TXO_CONN: now also SWD3.5 (Pin_5); no longer SWD3.7 (Pin_7)
- net GND: now also C6.1, C22.1, C23.1, C24.2; no longer C6.2
- net VCORE: now reaches C10.1, C5.1, U1.29 (VDDCORE)
Other:
- moved on the sheet: R10, R9
