File: mean-bean-pcb/mean-bean/d2-motherboard-pcb_mostly_rev1.kicad_sch (KiCad schematic)
At the start: 30 parts, among them J2 Conn_01x02_Male, J4 Conn_01x04_Male, U1 PIC32CM6408MC00032-I/PT

Commit message: rev2
Parts:
- removed C22, C25: 1uF, Capacitor_SMD:C_0603_1608Metric, symbol Device:C
- removed C23: 10uF, Capacitor_SMD:C_1206_3216Metric_Pad1.33x1.80mm_HandSolder, symbol Device:C
- removed C24: 22uF, Capacitor_SMD:C_0805_2012Metric_Pad1.18x1.45mm_HandSolder, symbol Device:C
- removed D2: LED, LED_SMD:LED_0603_1608Metric_Pad1.05x0.95mm_HandSolder, symbol Device:LED
- added J1: FTDI, Connector_PinHeader_2.54mm:PinHeader_1x06_P2.54mm_Vertical, symbol Connector:Conn_01x06_Male
- added J3: Conn_01x02_Male, Connector_PinHeader_2.54mm:PinHeader_1x02_P2.54mm_Vertical, symbol Connector:Conn_01x02_Male
- added SWD1: Conn_02x05_Odd_Even, Connector_PinHeader_1.27mm:PinHeader_2x05_P1.27mm_Vertical, symbol Connector_Generic:Conn_02x05_Odd_Even
- added TP1, TP2, TP5: TestPoint, Connector_PinHeader_2.54mm:PinHeader_1x01_P2.54mm_Vertical, symbol Connector:TestPoint
- C4: footprint Capacitor_THT:CP_Radial_D8.0mm_P3.50mm -> Capacitor_THT:CP_Radial_D5.0mm_P2.50mm
- C6: value 0.1uF -> 47uF; footprint Capacitor_SMD:C_0603_1608Metric -> Capacitor_THT:CP_Radial_D5.0mm_P2.50mm
- R16: value 330 -> 0
- renumbered SWD1 to SWD3
Connections:
- net +5V: now also C6.1, R16.1, SWD1.1 (Pin_1), TP1.1; no longer C6.2
- net CS1: now also TP5.1
- net FTDI_RXI_CONN: now also SWD3.5 (Pin_5), J1.2 (Pin_2); no longer SWD3.7 (Pin_7)
- net FTDI_TXO_CONN: now also SWD3.7 (Pin_7), J1.3 (Pin_3); no longer SWD3.5 (Pin_5)
- net GND: now also C6.2, J1.6 (Pin_6), SWD1.3 (Pin_3), SWD1.9 (Pin_9), TP2.1; no longer C6.1, R16.1
- net MISO: now also J3.1 (Pin_1)
- net RESET: now also SWD1.10 (Pin_10)
- net RX_FPORT_RX_SERCOM0: now also J3.2 (Pin_2); no longer U1.11 (PA08)
- net SWCLK: now also SWD1.4 (Pin_4)
- net SWDIO: now also SWD1.2 (Pin_2)
- net at R16.2: now also J1.4 (Pin_4)
- net VCORE: no longer names the net of C10.1, C5.1, U1.29 (VDDCORE)
- new net RX_FPORT_TX: U1.11 (PA08)
- no-connect marks 2 -> 0
Other:
- note added: "consider jumpering or even just switching"
- moved on the sheet: R10, R9
