File: mean-bean-pcb/mean-bean/mean-bean.kicad_pcb (KiCad board)
At the start: 4 copper layers, 49.5 x 38.8 mm, 48 parts, among them J1 Screw_Terminal_01x02, J2 Screw_Terminal_01x02, M3 Screw_Terminal_01x02, M4 Screw_Terminal_01x02, U1 PIC32CM6408MC00032-I/PT, U4 L9958, U5 L9958

Commit message: mean bean
Connections:
- U1 pad 14: PWM2 -> EN4
- U1 pad 23: EN4 -> CS3
- U1 pad 25: CS3 -> DIR3
- U1 pad 3: DIR3 -> unconnected-(U1-Pad3)
Routing:
- net EN4: track 43.9 -> 34.9 mm, vias 3 -> 2
- net DIR3: track 22.1 -> 13.9 mm
- net GND: track 125.8 -> 120.1 mm
- net PWM4: track 33.5 -> 37.7 mm
- net MISO: track 31.6 -> 28.0 mm, vias 3 -> 2
- net BATT: track 57.0 -> 56.1 mm
- net FTDI_TXO: track 30.1 -> 30.7 mm, vias 2 -> 3
- net FTDI_RXI: track 34.4 -> 35.0 mm, vias 2 -> 3
- net CS3: track 14.3 -> 13.7 mm
