File: mean-bean-pcb/mean-bean/mean-bean.kicad_sch (KiCad schematic)
At the start: 30 parts, among them J2 Conn_01x02_Male, J4 Conn_01x04_Male, U1 PIC32CM6408MC00032-I/PT

Commit message: rev2
Parts:
- removed J2: Conn_01x02_Male, Connector_PinHeader_2.54mm:PinHeader_1x02_P2.54mm_Vertical, symbol Connector:Conn_01x02_Male
- removed J4: Conn_01x04_Male, Connector_PinHeader_2.54mm:PinHeader_1x04_P2.54mm_Vertical, symbol Connector:Conn_01x04_Male
- added ESC1: BEC, Connector_PinHeader_2.54mm:PinHeader_1x03_P2.54mm_Vertical, symbol Connector:Conn_01x03_Male
- added J1, J2: Screw_Terminal_01x02, Connector_AMASS:AMASS_XT30U-M_1x02_P5.0mm_Vertical, symbol Connector:Screw_Terminal_01x02
- added R1: 0, Resistor_SMD:R_0603_1608Metric, symbol Device:R
Connections:
- net +5V: now also R1.2
- net BATT: now also J1.2 (Pin_2), J2.2 (Pin_2)
- net CS1: no longer U1.5 (PA04)
- net GND: now also ESC1.3 (Pin_3), J1.1 (Pin_1), J2.1 (Pin_1)
- net RX_FPORT_RX_SERCOM0: now also U1.5 (PA04); no longer U1.11 (PA08)
- new net: ESC1.2 (Pin_2), R1.1
- new net DSHOT_SERCOM2: ESC1.1 (Pin_1), U1.11 (PA08)
Other:
- removed sheet Channel1
- removed sheet Channel2
- moved on the sheet: BEC1, C24, C4

Commit message: mean bean
Connections:
- net CS3: now also U1.23 (PA24); no longer U1.25 (PA27)
- net DIR3: now also U1.25 (PA27); no longer U1.3 (PA02)
- net EN4: now also U1.14 (PA11); no longer U1.23 (PA24)
- net PWM2: no longer U1.14 (PA11)
Changed lines of the file:
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@@
-    )
-  )
-  (global_label "EN4" (shape input) (at 76.2 144.78 270) (fields_autoplaced)
-    (effects (font (size 1.27 1.27)) (justify right))
-    (property "Intersheet References" "${INTERSHEET_REFS}" (id 0) (at 76.2794 150.8821 90)
-      (effects (font (size 1.27 1.27)) (justify right) hide)
     )
   )
@@
     )
   )
-  (global_label "CS3" (shape input) (at 95.25 134.62 0) (fields_autoplaced)
-    (effects (font (size 1.27 1.27)) (justify left))
-    (property "Intersheet References" "${INTERSHEET_REFS}" (id 0) (at 101.3521 134.6994 0)
-      (effects (font (size 1.27 1.27)) (justify left) hide)
+  (global_label "CS3" (shape input) (at 76.2 144.78 270) (fields_autoplaced)
+    (effects (font (size 1.27 1.27)) (justify right))
+    (property "Intersheet References" "${INTERSHEET_REFS}" (id 0) (at 76.1206 150.8821 90)
+      (effects (font (size 1.27 1.27)) (justify right) hide)
     )
   )
@@
     )
   )
-  (global_label "DIR3" (shape input) (at 73.66 107.95 90) (fields_autoplaced)
-    (effects (font (size 1.27 1.27)) (justify left))
-    (property "Intersheet References" "${INTERSHEET_REFS}" (id 0) (at 73.7394 101.1826 90)
+  (global_label "EN4" (shape input) (at 48.26 130.81 180) (fields_autoplaced)
+    (effects (font (size 1.27 1.27)) (justify right))
+    (property "Intersheet References" "${INTERSHEET_REFS}" (id 0) (at 42.1579 130.8894 0)
+      (effects (font (size 1.27 1.27)) (justify right) hide)
+    )
+  )
+  (global_label "DIR3" (shape input) (at 95.25 134.62 0) (fields_autoplaced)
+    (effects (font (size 1.27 1.27)) (justify left))
+    (property "Intersheet References" "${INTERSHEET_REFS}" (id 0) (at 102.0174 134.6994 0)
       (effects (font (size 1.27 1.27)) (justify left) hide)
     )
@@
     )
   )
-  (global_label "PWM2" (shape input) (at 48.26 130.81 180) (fields_autoplaced)
-    (effects (font (size 1.27 1.27)) (justify right))
-    (property "Intersheet References" "${INTERSHEET_REFS}" (id 0) (at 40.4645 130.8894 0)
-      (effects (font (size 1.27 1.27)) (justify right) hide)
-    )
+  (global_label "PWM2" (shape input) (at 27.94 130.81 180) (fields_autoplaced)
+    (effects (font (size 1.27 1.27)) (justify right))
+    (property "Intersheet References" "${INTERSHEET_REFS}" (id 0) (at 20.1445 130.8894 0)
+      (effects (font (size 1.27 1.27)) (justify right) hide)
+    )
